File: V-00716-00.brd (EAGLE design)
At the start: 57 x 31.2 mm, 23 parts, among them Q1 16MHz, U1 ATMEGA32-16AU, X1 MINI-USB-32005-201

Commit message: v1.1.0.1
Routing:
- net GNDINT: track 127.1 -> 125.9 mm
- net PD0: track 20.7 -> 21.8 mm
- net N$1: track 52.0 -> 52.9 mm
- added copper zone on layer 1, net GNDINT
Other:
- board size 57 x 31.2 mm -> 63 x 39 mm
- board text added: "V-00716-00 Author: LN 11.12.2015"
