File: V-00716-02.sch (EAGLE design)
At the start: 20 parts, among them Q1 14.74MHz, U1 ATMEGA32U2-AU, X1 MINI-USB-32005-201

Commit message: v.2.1
Upravena verze + udelana verze 02 s upravy chyb
Parts:
- removed JUM5: S2G4_JUMP, #PaJa_konektory:S2G4_JUMP
- added JUM4: S2G2_JUMP, #PaJa_konektory:S2G2_JUMP
- added R10, R6: 0R, #PaJa_31:R_1206
- added R9: 10k, #PaJa_31:R_1206
Connections:
- net +5V: now also JUM42.1, JUM42.2, R9.2; no longer JUM52.1, JUM52.2, JUM52.3, JUM52.4
- net GNDINT: now also JUM41.1, JUM41.2, R10.1, R10.2, R6.1, R6.2; no longer JUM51.1, JUM51.2, JUM51.3, JUM51.4
- net RESET: now also R9.1
Other:
- note added: "+5V"
- note added: "10k"
- moved on the sheet: JUM3
